File: pcb/ESPlash/esplash.sch (EAGLE design)
At the start: 39 parts, among them IC1 ACS712, K1 SRD-05VDC-SL-C, K2 SRD-05VDC-SL-C, K3 SRD-05VDC-SL-C, K4 SRD-05VDC-SL-C, Q1 SMD-TRANSISTORS-PNP-25V-500MA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, Q2 SMD-TRANSISTORS-PNP-25V-500MA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, Q3 SMD-TRANSISTORS-PNP-25V-500MA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, Q4 SMD-TRANSISTORS-PNP-25V-500MA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, U1 ESP-WROOM-32

Commit message: update on Schematics of PCB
Parts:
- added C5, C6: (no value), fab:CAP-UNPOLARIZEDFAB
- added R12, R15: 10k, fab:RES-US1206
- added R13, R14: 100ohm, fab:RES-US1206
- added S1, S2: (no value), fab:6MM_SWITCH6MM_SWITCH
- added U$10, U$9: LED, fab:LED
- added U$6: ESP32DEVKITV1, ESP32-DEVKITV1:ESP32DEVKITV1
- added U$8: FTDI-SMD-HEADER, fab:FTDI-SMD-HEADER
- added Y1: ECS-.327-12.5-13X, ECS-.327-12.5-13X:ECS-.327-12.5-13X
Connections:
- removed net GPIO06: U1.CLK
- removed net GPIO08: U1.SD1
- removed net GPIO1: U1.IO0, U1.TXD0
- removed net GPIO10: U1.SD3
- removed net GPIO11: U1.CMD
- removed net GPIO13: U1.IO13
- removed net GPIO16: U1.IO16
- removed net GPIO2: U1.IO2, U1.RXD0
- removed net GPIO28: U1.IO17
- removed net GPIO32/DHT: R7.1, U1.IO32
- removed net GPIO33/PUMP_RELAY: R1.1, R11.2, U1.IO33
- removed net GPIO34: U1.IO34
- removed net GPIO36/CURRENT_SENSE: C4.1, IC1.VOUT, U1.SENSOR_VP
- removed net GPIO7: U1.SD0
- removed net GPIO9: U1.SD2
- new net 32K_XN: C6.2, R15.2, U$6.IO33, U1.IO33, Y1.1
- new net 32K_XP: C5.2, R15.1, U$6.IO32, U1.IO32, Y1.2
- new net GPIO02: R14.2, U$6.IO2, U1.IO2
- new net GPIO1/PROGRAMER: S2.P, S2.P1, U1.IO0
- new net GPIO1/TXD0: U$6.IO1, U$8.TXD, U1.TXD0
- new net GPIO13/PUMP_RELAY: R1.1, R11.2, U$6.IO13, U1.IO13
- new net GPIO16/CURRENT_SENSE: C4.1, IC1.VOUT, U$6.IO16, U1.IO16
- new net GPIO17: U$6.IO17, U1.IO17
- new net GPIO3/RXD0: U$6.IO3, U$8.RXD, U1.RXD0
- new net GPIO34/DHT: R7.1, U$6.IO34, U1.IO34
- new net GPIO36: U$6.VP-OI36, U1.SENSOR_VP
- new net GPIO5: U$6.IO5
- new net N$10: R14.1, U$10.A
- new net N$20: R13.1, U$9.A
- new net RESET: R12.2, S1.P, S1.P1, U$6.EN, U1.EN
- net 3.3V: now also R12.1, R13.2, U$6.3V3
- net 5V: now also U$6.VIN, U$8.VCC
- net GND: now also C5.1, C6.1, S1.S, S1.S1, S2.S, S2.S1, U$10.C, U$6.GND@1, U$6.GND@2, U$8.GND, U$9.C
- net GPIO12: now also U$6.IO12
- net GPIO14: now also U$6.IO14
- net GPIO15: now also U$6.IO15
- net GPIO18: now also U$6.IO18
- net GPIO19: now also U$6.IO19
- net GPIO21: now also U$6.IO21
- net GPIO22: now also U$6.IO22
- net GPIO23: now also U$6.IO23
- net GPIO25/VALVE_RELAY01: now also U$6.IO25
- net GPIO26/VALVE_RELAY02: now also U$6.IO26
- net GPIO27/VALVE_RELAY03: now also U$6.IO27
- net GPIO35/BATTVOLT: now also U$6.IO35
- net GPIO39: now also U$6.VN-IO39
- net GPIO4: now also U$6.IO4
Other:
- note added: "Buttons"
- note added: "Connectors"
- moved on the sheet: ACIN/OUT-1, ACIN/OUT-2, C1, C2, D1, D2, D3, D4, K1, K2, K3, K4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
