File: pcb/ESPlash/esplash.sch (EAGLE design)
At the start: 55 parts, among them IC1 ACS712, K1 SRD-05VDC-SL-C, K2 SRD-05VDC-SL-C, K3 SRD-05VDC-SL-C, K4 SRD-05VDC-SL-C, Q1 SMD-TRANSISTORS-PNP-25V-500MA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, Q2 SMD-TRANSISTORS-PNP-25V-500MA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, Q3 SMD-TRANSISTORS-PNP-25V-500MA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, Q4 SMD-TRANSISTORS-PNP-25V-500MA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, U1 ESP-WROOM-32, U2 EL817(S)(D)(TU)-V, U3 EL817(S)(D)(TU)-V, U4 EL817(S)(D)(TU)-V, U5 EL817(S)(D)(TU)-V, Y1 ECS-.327-12.5-13X

Commit message: pcb updates
Parts:
- added JP1, JP2: header2x6, pinhead:PINHD-2X3
- added POWER: 22-23-2021, con-molex:22-23-2021
- added R16: 100ohm, fab:RES-US1206
- added U$7: LED, fab:LED
- C3: value (none) -> 1nF
- C4: value (none) -> 0.1uF
- C5, C6: value (none) -> 15pf
- Q1, Q2, Q3, Q4: value SMD-TRANSISTORS-PNP-25V-500MA(SOT-23) -> BCX70SMD; device SMD-TRANSISTORS-PNP-25V-500MA_SOT-23_:SMD-TRANSISTORS-PNP-25V-500MA(SOT-23) -> transistor:BCX70SMD
- R10: value (none) -> 10K
- R11, R3, R6, R8: value (none) -> 100ohm
- R7: value (none) -> 1.2Mohm
- R9: value (none) -> 1.5Mohm
- S1: value (none) -> Reset
- S2: value (none) -> GPIO0 Button
- renumbered ACIN/OUT1 to VALVESOLENOID_01, ACIN/OUT2 to VALVESOLENOID_02, ACIN/OUT3 to VALVESOLENOID_03, U$8 to RTS
Connections:
- net 3.3V renamed 3V3
- net AMP_M/IN renamed AMP_METER/IN
- net AMP_M/OUT renamed AMP_METER/OUT
- net GPIO1/PROGRAMER renamed GPIO0
- net N$41 renamed ACIN
- net RESET renamed CHIP_PU
- removed net 5V: C4.2, D1.C, D2.C, D3.C, D4.C, IC1.VCC, K1.A1, K2.A1, K3.A1, K4.A1, R7.2, RTS.VCC, U$2.VIN, U2.CT, U3.CT, U4.CT, U5.CT
- new net N$27: JP2.1
- new net N$28: JP2.3
- new net N$29: R16.1, U$7.A
- new net RTS: RTS.RTS
- new net VCC: C4.2, D1.C, D2.C, D3.C, D4.C, IC1.VCC, K1.A1, K2.A1, K3.A1, K4.A1, POWER-1.S, R7.2, RTS.VCC, U$2.VIN, U2.CT, U3.CT, U4.CT, U5.CT
- net GND: now also C4.1, POWER-2.S, Q1.E, Q2.E, Q3.E, Q4.E, U$7.C; no longer Q1.C, Q2.C, Q3.C, Q4.C
- net GPIO05: now also JP1.4
- net GPIO12: now also JP2.4
- net GPIO14: now also JP2.2
- net GPIO16/CURRENT_SENSE: no longer C4.1
- net GPIO17: now also JP1.6
- net GPIO18: now also JP1.2
- net GPIO19: now also JP1.3
- net GPIO21: now also JP1.1
- net GPIO36: now also JP2.5
- net GPIO39: now also JP2.6
- net GPIO4: now also R16.2
- net PUMPRELAYSEGMENT: now also Q1.C; no longer Q1.E
- net RELAY1SEGMENT: now also Q2.C; no longer Q2.E
- net RELAY2SEGMENT: now also Q3.C; no longer Q3.E
- net RELAY3SEGMENT: now also Q4.C; no longer Q4.E
Other:
- moved on the sheet: C3, C4, IC1

Commit message: updates
Parts:
- added R17, R18, R19, R20: 220omh, fab:RES-US1206FAB
- R11, R3: value 100ohm -> 150ohm
Connections:
- removed net N$26: R10.2, U$6.DAT
- new net N$30: R17.2, U2.A
- new net N$31: R18.2, U3.A
- new net N$32: R19.2, U4.A
- new net N$33: R20.2, U5.A
- net 3V3: now also R10.2
- net GPIO13/PUMP_RELAY: now also R17.1; no longer U2.A
- net GPIO25/VALVE_RELAY01: now also R18.1; no longer U3.A
- net GPIO26/VALVE_RELAY02: now also R19.1; no longer U4.A
- net GPIO27/VALVE_RELAY03: now also R20.1; no longer U5.A
- net GPIO34/DHT: now also U$6.DAT
Other:
- moved on the sheet: ACIN/OUT-1, ACIN/OUT-2, D1, D2, D3, D4, K1, K2, K3, K4, Q1, Q2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
