File: pcb/ESPlash/esplash.brd (EAGLE design)
At the start: 160 x 100 mm, 28 parts, among them K1 SRD-05VDC-SL-C, K2 SRD-05VDC-SL-C, K3 SRD-05VDC-SL-C, K4 SRD-05VDC-SL-C, Q1 SMD-TRANSISTORS-PNP-25V-500MA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, Q2 SMD-TRANSISTORS-PNP-25V-500MA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, Q3 SMD-TRANSISTORS-PNP-25V-500MA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, Q4 SMD-TRANSISTORS-PNP-25V-500MA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, U1 ESP-WROOM-32

Commit message: update on Schematics of PCB
Parts:
- added C3, C4, C5, C6: (no value), fab:C1206FAB
- added IC1: ACS712, ACS712:SO08
- added R10, R11, R8, R9: (no value), fab:R1206FAB
- added R12, R15: 10k, fab:R1206
- added R13, R14: 100ohm, fab:R1206
- added S1, S2: (no value), fab:6MM_SWITCH
- added U$10, U$9: LED, fab:LED1206
- added U$3, U$4, U$5, U$7: LEDFAB1206, fab:LED1206FAB
- added U$6: ESP32DEVKITV1, ESP32-DEVKITV1:ESP32-DEVKITV1
- added U$8: FTDI-SMD-HEADER, fab:1X06SMD
- added Y1: ECS-.327-12.5-13X, ECS-.327-12.5-13X:XTAL_ECS-.327-12.5-13X
- moved U1 330.2 mm to (-240.0, -31.8)
- moved U$1 302.4 mm to (-214.6, 40.6), turned to 0 degrees
- moved C2 254.5 mm to (-142.2, 135.9)
- moved C1 251.0 mm to (-135.9, 135.9), turned to 0 degrees
- moved R6 188.5 mm to (-50.8, 142.2)
- moved R5 182.1 mm to (-45.7, 142.2), turned to 0 degrees
- moved R7 166.3 mm to (-55.9, 142.2), turned to 0 degrees
- moved U$2 140.1 mm to (-31.8, 124.5)
- moved D4 116.1 mm to (-29.2, 142.2)
- moved D2 116.1 mm to (-16.5, 142.2)
- moved D3 116.1 mm to (-22.9, 142.2)
- moved Q1 104.2 mm to (-135.9, 121.9)
- moved Q2 104.2 mm to (-157.5, 121.9)
- moved ACIN/OUT 77.8 mm to (-50.8, 123.2)
- moved NO1 77.8 mm to (-61.0, 123.2)
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Connections:
- removed net GPIO06: U1.20
- removed net GPIO08: U1.22
- removed net GPIO1: U1.25, U1.35
- removed net GPIO10: U1.18
- removed net GPIO11: U1.19
- removed net GPIO13: U1.16
- removed net GPIO16: U1.27
- removed net GPIO2: U1.24, U1.34
- removed net GPIO28: U1.28
- removed net GPIO32/DHT: R7.1, U1.8
- removed net GPIO33/PUMP_RELAY: R1.1, U1.9
- removed net GPIO34: U1.6
- removed net GPIO7: U1.21
- removed net GPIO9: U1.17
- new net 32K_XN: C6.2, R15.2, U$6.D33, U1.9, Y1.1
- new net 32K_XP: C5.2, R15.1, U$6.D32, U1.8, Y1.2
- new net DELETE: C3.2, IC1.6
- new net GPIO02: R14.2, U$6.D2, U1.24
- new net GPIO1/PROGRAMER: S2.1, S2.2, U1.25
- new net GPIO1/TXD0: U$6.D1, U$8.4, U1.35
- new net GPIO13/PUMP_RELAY: R1.1, R11.2, U$6.D13, U1.16
- new net GPIO16/CURRENT_SENSE: C4.1, IC1.7, U$6.D16, U1.27
- new net GPIO17: U$6.D17, U1.28
- new net GPIO3/RXD0: U$6.D3, U$8.5, U1.34
- new net GPIO34/DHT: R7.1, U$6.D34, U1.6
- new net GPIO5: U$6.D5
- new net N$10: R14.1, U$10.1
- new net N$2: R8.1, U$3.1
- new net N$20: R13.1, U$9.1
- new net N$5: R9.1, U$7.1
- new net N$7: R10.1, U$4.1
- new net N$8: R11.1, U$5.1
- new net RESET: R12.2, S1.1, S1.2, U$6.EN, U1.3
- net 3.3V: now also R12.1, R13.2, U$6.3V3
- net 5V: now also C4.2, IC1.8, U$6.VIN, U$8.3
- net AMP_M/IN: now also IC1.4
- net AMP_M/OUT: now also IC1.2
- net GND: now also C3.1, C5.1, C6.1, IC1.5, S1.3, S1.4, S2.3, S2.4, U$10.2, U$6.GND@1, U$6.GND@2, U$8.1, U$9.2
- net GPIO12: now also U$6.D12
- net GPIO14: now also U$6.D14
- net GPIO15: now also U$6.D15
- net GPIO18: now also U$6.D18
- net GPIO19: now also U$6.D19
- net GPIO21: now also U$6.D21
- net GPIO22: now also U$6.D22
- net GPIO23: now also U$6.D23
- net GPIO25/VALVE_RELAY01: now also R10.2, U$6.D25
- net GPIO26/VALVE_RELAY02: now also R9.2, U$6.D26
- net GPIO27/VALVE_RELAY03: now also R8.2, U$6.D27
- net GPIO35/BATTVOLT: now also U$6.D35
- net GPIO36: now also U$6.D36
- net GPIO39: now also U$6.D39
- net GPIO4: now also U$6.D4

Commit message: board
Parts:
- removed NO1, NO2, NO3: (no value), con-wago-500:W237-102
- removed U$7: LEDFAB1206, fab:LED1206FAB
- added ACIN/OUT1, ACIN/OUT2, ACIN/OUT3: (no value), con-wago-500:W237-102
- added U2, U3, U4, U5: EL817(S)(D)(TU)-V, EL817_S__D__TU_-V:SOIC254P1030X460-4N
- R3: value 1K -> (none)
- R5: value (none) -> 1K
- U$1: value MCP1700T-3302E/TT -> LEDFAB1206; device MCP1700T-3302E_TT:SOT95P237X112-3N -> fab:LED1206FAB
- U$2: value TEMP-HUM-SENSOR-DHT11 -> MCP1700T-3302E/TT; device diy-modules:TEMP-HUM-SENSOR-DHT11 -> MCP1700T-3302E_TT:SOT95P237X112-3N
- U$6: value ESP32DEVKITV1 -> TEMP-HUM-SENSOR-DHT11; device ESP32-DEVKITV1:ESP32-DEVKITV1 -> diy-modules:TEMP-HUM-SENSOR-DHT11
- moved R14 323.8 mm to (62.2, 43.2)
- moved U1 318.2 mm to (64.8, 59.7)
- moved U$10 313.8 mm to (62.2, 38.1)
- moved D1 279.7 mm to (92.7, 35.6)
- moved Y1 272.3 mm to (14.0, 58.4), turned to 180 degrees
- moved R15 272.0 mm to (20.3, 61.0), turned to 270 degrees
- moved C6 268.0 mm to (15.2, 53.3), turned to 90 degrees
- moved C5 264.3 mm to (12.7, 53.3), turned to 90 degrees
- moved R1 256.9 mm to (92.7, 44.5)
- moved U$1 254.4 mm to (39.4, 54.6)
- moved U$6 251.7 mm to (5.08, 34.3), turned to 90 degrees
- moved Q1 245.0 mm to (95.2, 40.6), turned to 270 degrees
- moved K4 234.2 mm to (63.5, 24.1), turned to 90 degrees
- moved IC1 225.0 mm to (81.3, 6.35), turned to 90 degrees
- moved K2 221.7 mm to (90.2, 21.6), turned to 90 degrees
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Connections:
- removed net C: D1.ANODE, D2.ANODE, D3.ANODE, D4.ANODE, K1.A2, K2.A2, K3.A2, K4.A2, Q1.2, Q2.2, Q3.2, Q4.2
- removed net GPIO5: U$6.D5
- removed net N$37: K1.NO, NO1.1
- removed net N$38: K1.COM, NO1.2
- removed net N$44: K3.NO, NO2.1
- removed net N$45: K3.COM, NO2.2
- removed net N$46: Q3.1, R3.2
- removed net N$48: K4.NO, NO3.1
- removed net N$49: K4.COM, NO3.2
- removed net N$50: Q4.1, R4.2
- removed net N$7 (its old number): R10.1, U$4.1
- new net N$13: R3.1, U$3.1
- new net N$14: R2.1, R3.2, U3.3
- new net N$15: ACIN/OUT2.2, K3.COM
- new net N$16: Q3.1, R4.2
- new net N$17: R8.1, U$4.1
- new net N$18: R4.1, R8.2, U4.3
- new net N$19: ACIN/OUT2.1, K3.NO
- new net N$20: ACIN/OUT3.2, K4.COM
- new net N$21: Q4.1, R5.2
- new net N$22: R6.1, U$1.1
- new net N$23: R5.1, R6.2, U5.3
- new net N$24: ACIN/OUT3.1, K4.NO
- new net N$26: R10.2, U$6.2
- new net PUMPRELAYSEGMENT: D1.ANODE, K2.A2, Q1.2
- new net RELAY1SEGMENT: D2.ANODE, K1.A2, Q2.2
- new net RELAY2SEGMENT: D3.ANODE, K3.A2, Q3.2
- new net RELAY3SEGMENT: D4.ANODE, K4.A2, Q4.2
- net 3.3V: now also U$2.2, U$6.1; no longer U$1.2, U$2.1, U$6.3V3
- net 32K_XN: no longer U$6.D33
- net 32K_XP: no longer U$6.D32
- net 5V: now also R7.2, U$2.3, U2.4, U3.4, U4.4, U5.4; no longer R5.2, U$1.3, U$6.VIN
- net AMP_M/IN: now also IC1.3
- net AMP_M/OUT: now also IC1.1
- net GND: now also R9.1, U$1.2, U$2.1, U$3.2, U$4.2, U$5.2, U$6.4, U2.2, U3.2, U4.2, U5.2; no longer R6.1, U$1.1, U$2.4, U$6.GND@1, U$6.GND@2
- net GPIO02: no longer U$6.D2
- net GPIO1/TXD0: no longer U$6.D1
- net GPIO12: no longer U$6.D12
- net GPIO13/PUMP_RELAY: now also U2.1; no longer R1.1, R11.2, U$6.D13
- net GPIO14: no longer U$6.D14
- net GPIO15: no longer U$6.D15
- net GPIO16/CURRENT_SENSE: no longer U$6.D16
- net GPIO17: no longer U$6.D17
- net GPIO18: no longer U$6.D18
- net GPIO19: no longer U$6.D19
- net GPIO21: no longer U$6.D21
- net GPIO22: no longer U$6.D22
- net GPIO23: no longer U$6.D23
- net GPIO25/VALVE_RELAY01: now also U3.1; no longer R10.2, R2.1, U$6.D25
- net GPIO26/VALVE_RELAY02: now also U4.1; no longer R3.1, R9.2, U$6.D26
- net GPIO27/VALVE_RELAY03: now also U5.1; no longer R4.1, R8.2, U$6.D27
- net GPIO3/RXD0: no longer U$6.D3
- net GPIO34/DHT: now also R10.1; no longer R7.1, U$6.D34
- net GPIO35/BATTVOLT: now also R7.1, R9.2; no longer R5.1, R6.2, U$6.D35
- net GPIO36: no longer U$6.D36
- net GPIO39: no longer U$6.D39
- net GPIO4: no longer U$6.D4
- net N$12: now also ACIN/OUT1.1, K1.NO; no longer R7.2, U$2.2
- net N$2: now also R1.1, R11.2, U2.3; no longer R8.1, U$3.1
- net N$5: now also ACIN/OUT1.2, K1.COM; no longer R9.1, U$7.1
- net RESET: no longer U$6.EN
Routing:
- net GND: track 0.00 -> 501.9 mm
- net 5V: track 0.00 -> 285.9 mm
- net 3.3V: track 0.00 -> 109.7 mm
- net GPIO35/BATTVOLT: track 0.00 -> 90.5 mm
- net RESET: track 0.00 -> 72.3 mm
- net GPIO34/DHT: track 0.00 -> 66.7 mm
- net GPIO16/CURRENT_SENSE: track 0.00 -> 56.0 mm
- net GPIO25/VALVE_RELAY01: track 0.00 -> 55.3 mm
- net GPIO13/PUMP_RELAY: track 0.00 -> 50.2 mm
- net 32K_XP: track 0.00 -> 49.6 mm
- net 32K_XN: track 0.00 -> 47.7 mm
- net RELAY3SEGMENT: track 0.00 -> 44.8 mm
- net RELAY2SEGMENT: track 0.00 -> 44.5 mm
- net RELAY1SEGMENT: track 0.00 -> 40.9 mm
- net GPIO26/VALVE_RELAY02: track 0.00 -> 32.3 mm
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Other:
- board size 160 x 100 mm -> 100 x 70 mm

Commit message: pcb updates
Parts:
- removed ACIN/OUT1, ACIN/OUT2, ACIN/OUT3: (no value), con-wago-500:W237-102
- removed U$8: FTDI-SMD-HEADER, fab:1X06SMD
- added JP1, JP2: header2x6, pinhead:2X03
- added POWER: 22-23-2021, con-molex:22-23-2021
- added R16: 100ohm, fab:R1206
- added RTS: FTDI-SMD-HEADER, fab:1X06SMD
- added U$7: LED, fab:LED1206
- added VALVESOLENOID_01, VALVESOLENOID_02, VALVESOLENOID_03: (no value), con-wago-500:W237-102
- C3: value (none) -> 1nF
- C4: value (none) -> 0.1uF
- C5, C6: value (none) -> 15pf
- Q1, Q2, Q3, Q4: value SMD-TRANSISTORS-PNP-25V-500MA(SOT-23) -> BCX70SMD; device SMD-TRANSISTORS-PNP-25V-500MA_SOT-23_:SOT-23 -> transistor:SOT23
- R10: value (none) -> 10K
- R11, R3, R6, R8: value (none) -> 100ohm
- R7: value (none) -> 1.2Mohm
- R9: value (none) -> 1.5Mohm
- S1: value (none) -> Reset
- S2: value (none) -> GPIO0 Button
- moved S1 42.7 mm to (46.2, 65.9), turned to 180 degrees
- moved R12 37.8 mm to (38.8, 65.2), turned to 270 degrees
- moved U$9 36.5 mm to (12.1, 40.1), turned to 45 degrees
- moved R9 35.9 mm to (24.4, 51.9), turned to 45 degrees
- moved C2 34.9 mm to (17.9, 42.7), turned to 135 degrees
- moved R10 34.8 mm to (34.4, 62.0)
- moved C1 34.7 mm to (20.6, 45.4), turned to 315 degrees
- moved U$2 34.7 mm to (23.3, 48.0), turned to 45 degrees
- moved R13 34.6 mm to (14.0, 38.3), turned to 45 degrees
- moved R7 31.4 mm to (27.3, 48.7), turned to 225 degrees
- moved Q3 30.6 mm to (41.6, 14.0)
- moved R4 30.2 mm to (40.4, 18.8), turned to 270 degrees
- moved Q4 30.1 mm to (62.1, 14.6)
- moved U5 30.0 mm to (63.7, 28.4)
- moved R5 29.7 mm to (61.4, 19.7), turned to 270 degrees
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Connections:
- net 3.3V renamed 3V3
- net AMP_M/IN renamed AMP_METER/IN
- net AMP_M/OUT renamed AMP_METER/OUT
- net GPIO1/PROGRAMER renamed GPIO0
- net N$41 renamed ACIN
- net RESET renamed CHIP_PU
- removed net 5V: C4.2, D1.CATHODE, D2.CATHODE, D3.CATHODE, D4.CATHODE, IC1.8, K1.A1, K2.A1, K3.A1, K4.A1, R7.2, U$2.3, U$8.3, U2.4, U3.4, U4.4, U5.4
- new net N$27: JP2.1
- new net N$28: JP2.3
- new net N$29: R16.1, U$7.1
- new net RTS: RTS.6
- new net VCC: C4.2, D1.CATHODE, D2.CATHODE, D3.CATHODE, D4.CATHODE, IC1.8, K1.A1, K2.A1, K3.A1, K4.A1, POWER.1, R7.2, RTS.3, U$2.3, U2.4, U3.4, U4.4, U5.4
- net GND: now also C4.1, POWER.2, Q1.2, Q2.2, Q3.2, Q4.2, RTS.1, U$7.2; no longer Q1.3, Q2.3, Q3.3, Q4.3, U$8.1
- net GPIO05: now also JP1.4
- net GPIO1/TXD0: now also RTS.4; no longer U$8.4
- net GPIO12: now also JP2.4
- net GPIO14: now also JP2.2
- net GPIO16/CURRENT_SENSE: no longer C4.1
- net GPIO17: now also JP1.6
- net GPIO18: now also JP1.2
- net GPIO19: now also JP1.3
- net GPIO21: now also JP1.1
- net GPIO3/RXD0: now also RTS.5; no longer U$8.5
- net GPIO36: now also JP2.5
- net GPIO39: now also JP2.6
- net GPIO4: now also R16.2
- net N$12: now also VALVESOLENOID_01.1; no longer ACIN/OUT1.1
- net N$15: now also VALVESOLENOID_02.2; no longer ACIN/OUT2.2
- net N$19: now also VALVESOLENOID_02.1; no longer ACIN/OUT2.1
- net N$20: now also VALVESOLENOID_03.2; no longer ACIN/OUT3.2
- net N$24: now also VALVESOLENOID_03.1; no longer ACIN/OUT3.1
- net N$5: now also VALVESOLENOID_01.2; no longer ACIN/OUT1.2
- net PUMPRELAYSEGMENT: now also Q1.3; no longer Q1.2
- net RELAY1SEGMENT: now also Q2.3; no longer Q2.2
- net RELAY2SEGMENT: now also Q3.3; no longer Q3.2
- net RELAY3SEGMENT: now also Q4.3; no longer Q4.2
Routing:
- net 5V: track 285.9 -> 0.00 mm
- net VCC: track 0.00 -> 256.4 mm
- net GPIO35/BATTVOLT: track 90.5 -> 33.8 mm
- net CHIP_PU: track 72.3 -> 16.6 mm
- net GPIO34/DHT: track 66.7 -> 17.2 mm
- net RELAY3SEGMENT: track 44.8 -> 5.47 mm
- net RELAY2SEGMENT: track 44.5 -> 5.41 mm
- net RELAY1SEGMENT: track 40.9 -> 5.40 mm
- net 3V3: track 109.7 -> 76.1 mm
- net GPIO27/VALVE_RELAY03: track 9.58 -> 43.0 mm
- net 32K_XN: track 47.7 -> 16.2 mm
- net 32K_XP: track 49.6 -> 18.6 mm
- net GPIO36: track 0.00 -> 23.1 mm
- net GND: track 501.9 -> 479.8 mm
- net GPIO39: track 0.00 -> 22.1 mm
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Other:
- board size 100 x 70 mm -> 101 x 71.1 mm
- board text added: "+"
- board text added: "GND"
- board text added: "Lucio"
- board text added: "RX"
- board text added: "TX"

Commit message: updates
Parts:
- added R17, R18, R19, R20: 220omh, fab:R1206FAB
- R11, R3: value 100ohm -> 150ohm
- moved R10 17.5 mm to (18.4, 54.7), turned to 135 degrees
Connections:
- removed net N$26: R10.2, U$6.2
- new net N$30: R17.2, U2.1
- new net N$31: R18.2, U3.1
- new net N$32: R19.2, U4.1
- new net N$33: R20.2, U5.1
- net 3V3: now also R10.2
- net GPIO13/PUMP_RELAY: now also R17.1; no longer U2.1
- net GPIO25/VALVE_RELAY01: now also R18.1; no longer U3.1
- net GPIO26/VALVE_RELAY02: now also R19.1; no longer U4.1
- net GPIO27/VALVE_RELAY03: now also R20.1; no longer U5.1
- net GPIO34/DHT: now also U$6.2
Routing:
- net GPIO34/DHT: track 17.2 -> 47.8 mm
- net N$26: track 27.5 -> 0.00 mm
- net GPIO13/PUMP_RELAY: track 41.7 -> 23.4 mm
- net N$30: track 0.00 -> 16.4 mm
- net GPIO25/VALVE_RELAY01: track 37.8 -> 31.6 mm
- net N$31: track 0.00 -> 5.81 mm
- net GPIO27/VALVE_RELAY03: track 43.0 -> 37.7 mm
- net N$32: track 0.00 -> 3.62 mm
- net N$33: track 0.00 -> 3.12 mm
- net GPIO26/VALVE_RELAY02: track 28.3 -> 26.1 mm
- net GPIO16/CURRENT_SENSE: track 70.4 -> 72.0 mm
- net VCC: track 256.4 -> 257.0 mm
Other:
- outline, holes or cut-outs redrawn
