File: pcb/ESPlash/esplashbpk.brd (EAGLE design)
At the start: 160 x 100 mm, 56 parts, among them IC1 ACS712, K1 SRD-05VDC-SL-C, K2 SRD-05VDC-SL-C, K3 SRD-05VDC-SL-C, K4 SRD-05VDC-SL-C, Q1 SMD-TRANSISTORS-PNP-25V-500MA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, Q2 SMD-TRANSISTORS-PNP-25V-500MA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, Q3 SMD-TRANSISTORS-PNP-25V-500MA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, Q4 SMD-TRANSISTORS-PNP-25V-500MA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, U1 ESP-WROOM-32, U2 EL817(S)(D)(TU)-V, U3 EL817(S)(D)(TU)-V, U4 EL817(S)(D)(TU)-V, U5 EL817(S)(D)(TU)-V, Y1 ECS-.327-12.5-13X

Commit message: pcb updates
Parts:
- removed ACIN/OUT1, ACIN/OUT2, ACIN/OUT3: (no value), con-wago-500:W237-102
- removed U$8: FTDI-SMD-HEADER, fab:1X06SMD
- added JP1, JP2: header2x6, pinhead:2X03
- added POWER: 22-23-2021, con-molex:22-23-2021
- added Q5, Q6: BCX70SMD, transistor:SOT23
- added R16: 100ohm, fab:R1206
- added R17, R18, R19: 10k, fab:R1206
- added RTS: FTDI-SMD-HEADER, fab:1X06SMD
- added VALVESOLENOID_01, VALVESOLENOID_02, VALVESOLENOID_03: (no value), con-wago-500:W237-102
- C3: value (none) -> 1nF
- C4: value (none) -> 0.1uF
- C5, C6: value (none) -> 15pf
- Q1, Q2, Q3, Q4: value SMD-TRANSISTORS-PNP-25V-500MA(SOT-23) -> BCX70SMD; device SMD-TRANSISTORS-PNP-25V-500MA_SOT-23_:SOT-23 -> transistor:SOT23
- R10: value (none) -> 10K
- R11, R3, R6, R8: value (none) -> 100ohm
- R5: value (none) -> 1K
- R7: value (none) -> 1.2Mohm
- R9: value 1K -> 1.5Mohm
- S1: value (none) -> Reset
- S2: value (none) -> GPIO0 Button
- U$1: value MCP1700T-3302E/TT -> LEDFAB1206; device MCP1700T-3302E_TT:SOT95P237X112-3N -> fab:LED1206FAB
- U$2: value TEMP-HUM-SENSOR-DHT11 -> MCP1700T-3302E/TT; device diy-modules:TEMP-HUM-SENSOR-DHT11 -> MCP1700T-3302E_TT:SOT95P237X112-3N
- U$6: value ESP32DEVKITV1 -> TEMP-HUM-SENSOR-DHT11; device ESP32-DEVKITV1:ESP32-DEVKITV1 -> diy-modules:TEMP-HUM-SENSOR-DHT11
- U$7: value LEDFAB1206 -> LED; device fab:LED1206FAB -> fab:LED1206
- moved U$1 270.2 mm to (55.4, 31.8)
- moved ACIN/OUT 267.8 mm to (89.8, 6.35)
- moved R11 256.6 mm to (79.1, 28.9)
- moved S2 254.0 mm to (69.3, 41.0), turned to 270 degrees
- moved K4 234.2 mm to (61.9, 19.1), flipped to the bottom
- moved C4 228.1 mm to (75.9, 3.81), turned to 270 degrees
- moved U$4 226.9 mm to (35.2, 31.8)
- moved R5 223.6 mm to (61.4, 19.7), turned to 270 degrees
- moved C3 221.0 mm to (75.9, 8.89), turned to 270 degrees
- moved R6 218.2 mm to (55.3, 28.4)
- moved K2 217.5 mm to (84.8, 19.1), flipped to the bottom
- moved S1 215.0 mm to (46.2, 65.9), turned to 180 degrees
- moved R8 210.0 mm to (35.2, 27.9)
- moved U$10 209.9 mm to (59.4, 44.5), turned to 90 degrees
- moved R14 207.6 mm to (63.2, 44.5), turned to 90 degrees
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Connections:
- net N$41 renamed ACIN
- removed net 3.3V: C1.2, C2.1, R12.1, R13.2, U$1.2, U$2.1, U$6.3V3, U1.2
- removed net 5V: C4.2, D1.CATHODE, D2.CATHODE, D3.CATHODE, D4.CATHODE, IC1.8, K1.A1, K2.A1, K3.A1, K4.A1, R5.2, U$1.3, U$6.VIN, U$8.3, U2.4, U3.4, U4.4, U5.4
- removed net AMP_M/IN: IC1.4, K1.NO, K2.NO, K3.NO, K4.NO
- removed net AMP_M/OUT: ACIN/OUT.1, ACIN/OUT1.1, ACIN/OUT2.1, ACIN/OUT3.1, IC1.2
- removed net C: D3.ANODE, D4.ANODE, K3.A2, K4.A2, Q3.2, Q4.2
- removed net GPIO1/PROGRAMER: S2.1, S2.2, U1.25
- removed net GPIO5: U$6.D5
- removed net PUMPRELAY: D1.ANODE, K2.A2, Q1.2
- removed net RELAY2: D2.ANODE, K1.A2, Q2.2
- removed net RESET: R12.2, S1.1, S1.2, U$6.EN, U1.3
- new net 3V3: C1.2, C2.1, R12.1, R13.2, R17.1, U$2.2, U$6.1, U1.2
- new net AMP_METER/IN: IC1.3, IC1.4, K2.NO
- new net AMP_METER/OUT: ACIN/OUT.1, IC1.1, IC1.2
- new net CHIP_PU: Q6.3, R12.2, S1.1, S1.2, U1.3
- new net DTR: Q5.2, R19.2
- new net GPIO0: Q5.3, R17.2, S2.1, S2.2, U1.25
- new net N$20: K4.COM, VALVESOLENOID_03.2
- new net N$24: K4.NO, VALVESOLENOID_03.1
- new net N$26: R10.2, U$6.2
- new net N$27: JP2.1
- new net N$28: JP2.3
- new net N$29: R16.1, U$7.1
- new net N$31: Q5.1, R18.1
- new net N$34: Q6.1, R19.1
- new net PUMPRELAYSEGMENT: D1.ANODE, K2.A2, Q1.3
- new net RELAY1SEGMENT: D2.ANODE, K1.A2, Q2.3
- new net RELAY2SEGMENT: D3.ANODE, K3.A2, Q3.3
- new net RELAY3SEGMENT: D4.ANODE, K4.A2, Q4.3
- new net RTS: Q6.2, R18.2, RTS.6
- new net VCC: C4.2, D1.CATHODE, D2.CATHODE, D3.CATHODE, D4.CATHODE, IC1.8, K1.A1, K2.A1, K3.A1, K4.A1, POWER.1, R7.2, RTS.3, U$2.3, U2.4, U3.4, U4.4, U5.4
- net 32K_XN: no longer U$6.D33
- net 32K_XP: no longer U$6.D32
- net GND: now also C4.1, POWER.2, Q1.2, Q2.2, Q3.2, Q4.2, R9.1, RTS.1, U$1.2, U$2.1, U$6.4; no longer Q1.3, Q2.3, Q3.3, Q4.3, R6.1, U$1.1, U$2.4, U$6.GND@1, U$6.GND@2, U$8.1
- net GPIO02: no longer U$6.D2
- net GPIO05: now also JP1.4
- net GPIO1/TXD0: now also RTS.4; no longer U$6.D1, U$8.4
- net GPIO12: now also JP2.4; no longer U$6.D12
- net GPIO13/PUMP_RELAY: no longer U$6.D13
- net GPIO14: now also JP2.2; no longer U$6.D14
- net GPIO15: no longer U$6.D15
- net GPIO16/CURRENT_SENSE: no longer C4.1, U$6.D16
- net GPIO17: now also JP1.6; no longer U$6.D17
- net GPIO18: now also JP1.2; no longer U$6.D18
- net GPIO19: now also JP1.3; no longer U$6.D19
- net GPIO21: now also JP1.1; no longer U$6.D21
- net GPIO22: no longer U$6.D22
- net GPIO23: no longer U$6.D23
- net GPIO25/VALVE_RELAY01: no longer U$6.D25
- net GPIO26/VALVE_RELAY02: no longer U$6.D26
- net GPIO27/VALVE_RELAY03: no longer U$6.D27
- net GPIO3/RXD0: now also RTS.5; no longer U$6.D3, U$8.5
- net GPIO34/DHT: now also R10.1; no longer R7.1, U$6.D34
- net GPIO35/BATTVOLT: now also R7.1, R9.2; no longer R5.1, R6.2, U$6.D35
- net GPIO36: now also JP2.5; no longer U$6.D36
- net GPIO39: now also JP2.6; no longer U$6.D39
- net GPIO4: now also R16.2; no longer U$6.D4
- net N$12: now also K1.NO, VALVESOLENOID_01.1; no longer R7.2, U$2.2
- net N$15: now also VALVESOLENOID_02.2; no longer ACIN/OUT2.2
- net N$19: now also K3.NO, VALVESOLENOID_02.1; no longer ACIN/OUT3.2, K4.COM
- net N$21: now also R5.2; no longer R9.2
- net N$22: now also R6.1, U$1.1; no longer R10.1, U$7.1
- net N$23: now also R5.1, R6.2; no longer R10.2, R9.1
- net N$5: now also VALVESOLENOID_01.2; no longer ACIN/OUT1.2
Routing:
- net GND: track 0.00 -> 479.8 mm
- net VCC: track 0.00 -> 255.7 mm
- net 3V3: track 0.00 -> 76.1 mm
- net GPIO16/CURRENT_SENSE: track 0.00 -> 70.4 mm
- net GPIO27/VALVE_RELAY03: track 0.00 -> 43.0 mm
- net GPIO13/PUMP_RELAY: track 0.00 -> 41.7 mm
- net GPIO25/VALVE_RELAY01: track 0.00 -> 37.8 mm
- net GPIO35/BATTVOLT: track 0.00 -> 33.8 mm
- net GPIO26/VALVE_RELAY02: track 0.00 -> 28.3 mm
- net N$26: track 0.00 -> 27.5 mm
- net GPIO36: track 0.00 -> 23.1 mm
- net GPIO0: track 0.00 -> 22.1 mm
- net GPIO39: track 0.00 -> 22.1 mm
- net GPIO14: track 0.00 -> 19.8 mm
- net 32K_XP: track 0.00 -> 18.6 mm
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Other:
- board size 160 x 100 mm -> 101 x 71.1 mm
- board text added: "+"
- board text added: "C:/Users/lpgn/Desktop/123.bmp"
- board text added: "GND"
- board text added: "Lucio"
- board text added: "RX"
- board text added: "TX"
