File: pcb/ESPlash/esplashbpk.sch (EAGLE design)
At the start: 45 parts, among them IC1 ACS712, K1 SRD-05VDC-SL-C, K2 SRD-05VDC-SL-C, K3 SRD-05VDC-SL-C, K4 SRD-05VDC-SL-C, Q1 SMD-TRANSISTORS-PNP-25V-500MA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, Q2 SMD-TRANSISTORS-PNP-25V-500MA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, Q3 SMD-TRANSISTORS-PNP-25V-500MA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, Q4 SMD-TRANSISTORS-PNP-25V-500MA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, U1 ESP-WROOM-32, U2 EL817(S)(D)(TU)-V, U3 EL817(S)(D)(TU)-V, U4 EL817(S)(D)(TU)-V, U5 EL817(S)(D)(TU)-V

Commit message: board
Parts:
- added C5, C6: (no value), fab:CAP-UNPOLARIZEDFAB
- added R10: (no value), fab:RES-US1206FAB
- added R12, R15: 10k, fab:RES-US1206
- added S1, S2: (no value), fab:6MM_SWITCH6MM_SWITCH
- added U$6: ESP32DEVKITV1, ESP32-DEVKITV1:ESP32DEVKITV1
- added U$7: LEDFAB1206, fab:LEDFAB1206
- added U$8: FTDI-SMD-HEADER, fab:FTDI-SMD-HEADER
- added Y1: ECS-.327-12.5-13X, ECS-.327-12.5-13X:ECS-.327-12.5-13X
- R5: value 1K -> (none)
- R9: value (none) -> 1K
- U$1: value LEDFAB1206 -> MCP1700T-3302E/TT; device fab:LEDFAB1206 -> MCP1700T-3302E_TT:MCP1700T-3302E/TT
- U$2: value MCP1700T-3302E/TT -> TEMP-HUM-SENSOR-DHT11; device MCP1700T-3302E_TT:MCP1700T-3302E/TT -> diy-modules:TEMP-HUM-SENSOR-DHT11
Connections:
- net PUMPRELAYSEGMENT renamed PUMPRELAY
- net RELAY1SEGMENT renamed RELAY2
- removed net N$19 (its old number): ACIN/OUT2-1.KL, K3.NO
- removed net N$24: ACIN/OUT3-1.KL, K4.NO
- removed net RELAY2SEGMENT: D3.A, K3.A2, Q3.E
- removed net RELAY3SEGMENT: D4.A, K4.A2, Q4.E
- new net C: D3.A, D4.A, K3.A2, K4.A2, Q3.E, Q4.E
- new net GPIO5: U$6.IO5
- net 3.3V: now also R12.1, U$1.VOUT, U$2.VDD, U$6.3V3; no longer U$2.VOUT
- net 32K_XN: now also C6.2, R15.2, U$6.IO33, Y1.1
- net 32K_XP: now also C5.2, R15.1, U$6.IO32, Y1.2
- net 5V: now also R5.2, U$1.VIN, U$6.VIN, U$8.VCC; no longer R7.2, U$2.VIN
- net AMP_M/IN: now also K1.NO, K3.NO, K4.NO; no longer IC1.I-_0
- net AMP_M/OUT: now also ACIN/OUT1-1.KL, ACIN/OUT2-1.KL, ACIN/OUT3-1.KL; no longer IC1.I+_0
- net GND: now also C5.1, C6.1, R6.1, S1.S, S1.S1, S2.S, S2.S1, U$1.GND, U$6.GND@1, U$6.GND@2, U$7.C, U$8.GND; no longer R9.1, U$1.C
- net GPIO02: now also U$6.IO2
- net GPIO1/PROGRAMER: now also S2.P, S2.P1
- net GPIO1/TXD0: now also U$6.IO1, U$8.TXD
- net GPIO12: now also U$6.IO12
- net GPIO13/PUMP_RELAY: now also U$6.IO13
- net GPIO14: now also U$6.IO14
- net GPIO15: now also U$6.IO15
- net GPIO16/CURRENT_SENSE: now also U$6.IO16
- net GPIO17: now also U$6.IO17
- net GPIO18: now also U$6.IO18
- net GPIO19: now also U$6.IO19
- net GPIO21: now also U$6.IO21
- net GPIO22: now also U$6.IO22
- net GPIO23: now also U$6.IO23
- net GPIO25/VALVE_RELAY01: now also U$6.IO25
- net GPIO26/VALVE_RELAY02: now also U$6.IO26
- net GPIO27/VALVE_RELAY03: now also U$6.IO27
- net GPIO3/RXD0: now also U$6.IO3, U$8.RXD
- net GPIO34/DHT: now also R7.1, U$6.IO34
- net GPIO35/BATTVOLT: now also R5.1, R6.2, U$6.IO35; no longer R7.1, R9.2
- net GPIO36: now also U$6.VP-OI36
- net GPIO39: now also U$6.VN-IO39
- net GPIO4: now also U$6.IO4
- net N$12: now also R7.2, U$2.DAT; no longer ACIN/OUT1-1.KL, K1.NO
- net N$21: now also R9.2; no longer R5.2
- net N$22: now also R10.1, U$7.A; no longer R6.1, U$1.A
- net N$23: now also R10.2, R9.1; no longer R5.1, R6.2
- net RESET: now also R12.2, S1.P, S1.P1, U$6.EN
Other:
- moved on the sheet: ACIN/OUT-1, ACIN/OUT-2, ACIN/OUT2-1, ACIN/OUT2-2, ACIN/OUT3-1, ACIN/OUT3-2, C1, C2, C3, C4, D3, D4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

Commit message: pcb updates
Parts:
- removed ACIN/OUT2, ACIN/OUT3: (no value), con-wago-500:W237-102
- added JP1, JP2: header2x6, pinhead:PINHD-2X3
- added POWER: 22-23-2021, con-molex:22-23-2021
- added Q5, Q6: BCX70SMD, transistor:BCX70SMD
- added R16: 100ohm, fab:RES-US1206
- added R17, R18, R19: 10k, fab:RES-US1206
- added VALVESOLENOID_02, VALVESOLENOID_03: (no value), con-wago-500:W237-102
- C3: value (none) -> 1nF
- C4: value (none) -> 0.1uF
- C5, C6: value (none) -> 15pf
- Q1, Q2, Q3, Q4: value SMD-TRANSISTORS-PNP-25V-500MA(SOT-23) -> BCX70SMD; device SMD-TRANSISTORS-PNP-25V-500MA_SOT-23_:SMD-TRANSISTORS-PNP-25V-500MA(SOT-23) -> transistor:BCX70SMD
- R10: value (none) -> 10K
- R11, R3, R6, R8: value (none) -> 100ohm
- R5: value (none) -> 1K
- R7: value (none) -> 1.2Mohm
- R9: value 1K -> 1.5Mohm
- S1: value (none) -> Reset
- S2: value (none) -> GPIO0 Button
- U$1: value MCP1700T-3302E/TT -> LEDFAB1206; device MCP1700T-3302E_TT:MCP1700T-3302E/TT -> fab:LEDFAB1206
- U$2: value TEMP-HUM-SENSOR-DHT11 -> MCP1700T-3302E/TT; device diy-modules:TEMP-HUM-SENSOR-DHT11 -> MCP1700T-3302E_TT:MCP1700T-3302E/TT
- U$6: value ESP32DEVKITV1 -> TEMP-HUM-SENSOR-DHT11; device ESP32-DEVKITV1:ESP32DEVKITV1 -> diy-modules:TEMP-HUM-SENSOR-DHT11
- U$7: value LEDFAB1206 -> LED; device fab:LEDFAB1206 -> fab:LED
- renumbered ACIN/OUT1 to VALVESOLENOID_01, U$8 to RTS
Connections:
- net N$41 renamed ACIN
- removed net 3.3V: C1.2, C2.1, R12.1, R13.2, U$1.VOUT, U$2.VDD, U$6.3V3, U1.3V3
- removed net 5V: C4.2, D1.C, D2.C, D3.C, D4.C, IC1.VCC, K1.A1, K2.A1, K3.A1, K4.A1, R5.2, RTS.VCC, U$1.VIN, U$6.VIN, U2.CT, U3.CT, U4.CT, U5.CT
- removed net AMP_M/IN: IC1.I-_1, K1.NO, K2.NO, K3.NO, K4.NO
- removed net AMP_M/OUT: ACIN/OUT-1.KL, ACIN/OUT2-1.KL, ACIN/OUT3-1.KL, IC1.I+_1, VALVESOLENOID_01-1.KL
- removed net C: D3.A, D4.A, K3.A2, K4.A2, Q3.E, Q4.E
- removed net GPIO1/PROGRAMER: S2.P, S2.P1, U1.IO0
- removed net GPIO5: U$6.IO5
- removed net PUMPRELAY: D1.A, K2.A2, Q1.E
- removed net RELAY2: D2.A, K1.A2, Q2.E
- removed net RESET: R12.2, S1.P, S1.P1, U$6.EN, U1.EN
- new net 3V3: C1.2, C2.1, R12.1, R13.2, R17.1, U$2.VOUT, U$6.VDD, U1.3V3
- new net AMP_METER/IN: IC1.I-_0, IC1.I-_1, K2.NO
- new net AMP_METER/OUT: ACIN/OUT-1.KL, IC1.I+_0, IC1.I+_1
- new net CHIP_PU: Q6.C, R12.2, S1.P, S1.P1, U1.EN
- new net DTR: Q5.E, R19.2
- new net GPIO0: Q5.C, R17.2, S2.P, S2.P1, U1.IO0
- new net N$20: K4.COM, VALVESOLENOID_03-2.KL
- new net N$24: K4.NO, VALVESOLENOID_03-1.KL
- new net N$26: R10.2, U$6.DAT
- new net N$27: JP2.1
- new net N$28: JP2.3
- new net N$29: R16.1, U$7.A
- new net N$31: Q5.B, R18.1
- new net N$34: Q6.B, R19.1
- new net PUMPRELAYSEGMENT: D1.A, K2.A2, Q1.C
- new net RELAY1SEGMENT: D2.A, K1.A2, Q2.C
- new net RELAY2SEGMENT: D3.A, K3.A2, Q3.C
- new net RELAY3SEGMENT: D4.A, K4.A2, Q4.C
- new net RTS: Q6.E, R18.2, RTS.RTS
- new net VCC: C4.2, D1.C, D2.C, D3.C, D4.C, IC1.VCC, K1.A1, K2.A1, K3.A1, K4.A1, POWER-1.S, R7.2, RTS.VCC, U$2.VIN, U2.CT, U3.CT, U4.CT, U5.CT
- net 32K_XN: no longer U$6.IO33
- net 32K_XP: no longer U$6.IO32
- net GND: now also C4.1, POWER-2.S, Q1.E, Q2.E, Q3.E, Q4.E, R9.1, U$1.C, U$6.GND; no longer Q1.C, Q2.C, Q3.C, Q4.C, R6.1, U$1.GND, U$6.GND@1, U$6.GND@2
- net GPIO02: no longer U$6.IO2
- net GPIO05: now also JP1.4
- net GPIO1/TXD0: no longer U$6.IO1
- net GPIO12: now also JP2.4; no longer U$6.IO12
- net GPIO13/PUMP_RELAY: no longer U$6.IO13
- net GPIO14: now also JP2.2; no longer U$6.IO14
- net GPIO15: no longer U$6.IO15
- net GPIO16/CURRENT_SENSE: no longer C4.1, U$6.IO16
- net GPIO17: now also JP1.6; no longer U$6.IO17
- net GPIO18: now also JP1.2; no longer U$6.IO18
- net GPIO19: now also JP1.3; no longer U$6.IO19
- net GPIO21: now also JP1.1; no longer U$6.IO21
- net GPIO22: no longer U$6.IO22
- net GPIO23: no longer U$6.IO23
- net GPIO25/VALVE_RELAY01: no longer U$6.IO25
- net GPIO26/VALVE_RELAY02: no longer U$6.IO26
- net GPIO27/VALVE_RELAY03: no longer U$6.IO27
- net GPIO3/RXD0: no longer U$6.IO3
- net GPIO34/DHT: now also R10.1; no longer R7.1, U$6.IO34
- net GPIO35/BATTVOLT: now also R7.1, R9.2; no longer R5.1, R6.2, U$6.IO35
- net GPIO36: now also JP2.5; no longer U$6.VP-OI36
- net GPIO39: now also JP2.6; no longer U$6.VN-IO39
- net GPIO4: now also R16.2; no longer U$6.IO4
- net N$12: now also K1.NO, VALVESOLENOID_01-1.KL; no longer R7.2, U$2.DAT
- net N$15: now also VALVESOLENOID_02-2.KL; no longer ACIN/OUT2-2.KL
- net N$19: now also K3.NO, VALVESOLENOID_02-1.KL; no longer ACIN/OUT3-2.KL, K4.COM
- net N$21: now also R5.2; no longer R9.2
- net N$22: now also R6.1, U$1.A; no longer R10.1, U$7.A
- net N$23: now also R5.1, R6.2; no longer R10.2, R9.1
Other:
- moved on the sheet: ACIN/OUT-1, ACIN/OUT-2, C1, C2, C3, C4, D3, D4, IC1, K3, K4, R10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
