File: pcb/ESPlash/1.0/esplash.brd (EAGLE design)
At the start: 101 x 71.1 mm, 64 parts, among them IC1 ACS712, K1 SRD-05VDC-SL-C, K2 SRD-05VDC-SL-C, K3 SRD-05VDC-SL-C, K4 SRD-05VDC-SL-C, Q1 BCX70SMD, Q2 BCX70SMD, Q3 BCX70SMD, Q4 BCX70SMD, U1 ESP-WROOM-32, U2 EL817(S)(D)(TU)-V, U3 EL817(S)(D)(TU)-V, U4 EL817(S)(D)(TU)-V, U5 EL817(S)(D)(TU)-V, Y1 ECS-.327-12.5-13X

Commit message: update
Parts:
- moved R2 173.0 mm to (-0.43, -41.1)
- moved Q2 172.8 mm to (-2.63, -45.3)
- moved D2 172.2 mm to (2.22, -39.8)
- moved D3 172.2 mm to (24.5, -39.9)
- moved U$3 171.7 mm to (-4.78, -41.1)
- moved U$4 171.7 mm to (16.9, -42.4)
- moved K1 171.5 mm to (-2.47, -37.0)
- moved K3 171.5 mm to (19.5, -37.3)
- moved Q3 171.5 mm to (19.5, -46.2)
- moved R18 171.5 mm to (3.83, -25.5)
- moved R19 171.5 mm to (26.0, -26.8)
- moved R3 171.5 mm to (-3.27, -35.6)
- moved R4 171.5 mm to (20.8, -41.4)
- moved R8 171.5 mm to (18.2, -37.3)
- moved U3 171.5 mm to (-0.47, -28.4)
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Routing:
- net GND: track 550.1 -> 265.7 mm
- net VCC: track 421.1 -> 141.5 mm
- net GPIO25/VALVE_RELAY01: track 95.9 -> 4.18 mm
- net GPIO26/VALVE_RELAY02: track 88.9 -> 3.83 mm
- net GPIO27/VALVE_RELAY03: track 73.3 -> 3.03 mm
- net GPIO16/CURRENT_SENSE: track 72.0 -> 45.0 mm
- net GPIO13/PUMP_RELAY: track 23.4 -> 3.88 mm
- net N$30: track 16.4 -> 6.54 mm
- net N$23: track 10.2 -> 6.46 mm
- net N$24: track 12.0 -> 15.0 mm
- net N$33: track 3.12 -> 5.56 mm
- net RELAY3SEGMENT: track 5.47 -> 7.88 mm
- net N$12: track 16.6 -> 14.5 mm
- net N$14: track 5.32 -> 7.05 mm
- net RELAY2SEGMENT: track 8.36 -> 10.0 mm
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