File: pcb/esplash.brd (EAGLE design)
At the start: 101 x 71.1 mm, 64 parts, among them IC1 ACS712, K1 SRD-05VDC-SL-C, K2 SRD-05VDC-SL-C, K3 SRD-05VDC-SL-C, K4 SRD-05VDC-SL-C, Q1 BCX70SMD, Q2 BCX70SMD, Q3 BCX70SMD, Q4 BCX70SMD, U1 ESP-WROOM-32, U2 EL817(S)(D)(TU)-V, U3 EL817(S)(D)(TU)-V, U4 EL817(S)(D)(TU)-V, U5 EL817(S)(D)(TU)-V, Y1 ECS-.327-12.5-13X

Commit message: updates
Parts:
- R17, R18, R19, R20: value 220omh -> 120omh
