File: pcb/esplash.sch (EAGLE design)
At the start: 64 parts, among them IC1 ACS712, K1 SRD-05VDC-SL-C, K2 SRD-05VDC-SL-C, K3 SRD-05VDC-SL-C, K4 SRD-05VDC-SL-C, Q1 BCX70SMD, Q2 BCX70SMD, Q3 BCX70SMD, Q4 BCX70SMD, U1 ESP-WROOM-32, U2 EL817(S)(D)(TU)-V, U3 EL817(S)(D)(TU)-V, U4 EL817(S)(D)(TU)-V, U5 EL817(S)(D)(TU)-V, Y1 ECS-.327-12.5-13X

Commit message: updates
Parts:
- R17, R18, R19, R20: value 220omh -> 120omh
Changed lines of the file:
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@@
 <part name="GND16" library="supply1" library_urn="urn:adsk.eagle:library:371" deviceset="GND" device=""/>
 <part name="R2" library="fab" deviceset="RES-US" device="1206FAB" value="1K"/>
-<part name="R17" library="fab" deviceset="RES-US" device="1206FAB" value="220omh"/>
-<part name="R18" library="fab" deviceset="RES-US" device="1206FAB" value="220omh"/>
-<part name="R19" library="fab" deviceset="RES-US" device="1206FAB" value="220omh"/>
-<part name="R20" library="fab" deviceset="RES-US" device="1206FAB" value="220omh"/>
+<part name="R17" library="fab" deviceset="RES-US" device="1206FAB" value="120omh"/>
+<part name="R18" library="fab" deviceset="RES-US" device="1206FAB" value="120omh"/>
+<part name="R19" library="fab" deviceset="RES-US" device="1206FAB" value="120omh"/>
+<part name="R20" library="fab" deviceset="RES-US" device="1206FAB" value="120omh"/>
 </parts>
 <sheets>
