File: pcb/0.1/esplashbpk.sch (EAGLE design)
At the start: 57 parts, among them Q5 BCX70SMD, Q6 BCX70SMD, U1 ESP-WROOM-32, Y1 ECS-.327-12.5-13X

Commit message: PCB changes
Parts:
- removed GND1, SC_00, SC_01, SC_02, SC_03, SC_04, SC_05, SC_06, SC_07, SC_08: SC, con-wago-500:W237-103
- removed R21, R22: 10k, fab:RES-US1206
- removed U$11, U$12, U$13, U$14, U$15, U$16, U$8: LED, fab:LED
- added ACIN/OUT, VALVESOLENOID_01, VALVESOLENOID_02, VALVESOLENOID_03: (no value), con-wago-500:W237-102
- added C3: 1nF, fab:CAP-UNPOLARIZEDFAB
- added C4: 0.1uF, fab:CAP-UNPOLARIZEDFAB
- added D1, D2, D3, D4: (no value), fab:DIODESOD123
- added IC1: ACS712, ACS712:ACS712
- added JP1, JP2: header2x6, pinhead:PINHD-2X3
- added K1, K2, K3, K4: SRD-05VDC-SL-C, SRD-05VDC-SL-C:SRD-05VDC-SL-C
- added Q1, Q2, Q3, Q4: BCX70SMD, transistor:BCX70SMD
- added R3: 100ohm, fab:RES-US1206FAB
- added U$4: LEDFAB1206, fab:LEDFAB1206
- added U2, U3, U4, U5: EL817(S)(D)(TU)-V, EL817_S__D__TU_-V:EL817(S)(D)(TU)-V
- R1, R2, R4, R5: value 100ohm -> 1K; device fab:RES-US1206 -> fab:RES-US1206FAB
- R11, R6, R8: device fab:RES-US1206 -> fab:RES-US1206FAB
- R17, R18, R19: value 100ohm -> 10k
- U$1, U$3, U$5: value LED -> LEDFAB1206; device fab:LED -> fab:LEDFAB1206
Connections:
- removed net GPIO05/VALVE_RELAY07: R18.2, SC_07-3.KL, U1.IO5
- removed net GPIO17/VALVE_RELAY08: R19.2, SC_08-3.KL, U1.IO17
- removed net GPIO18/VALVE_RELAY06: R17.2, SC_06-3.KL, U1.IO18
- removed net GPIO19/VALVE_RELAY05: R16.2, SC_05-3.KL, U1.IO19
- removed net GPIO21/VALVE_RELAY04: R1.2, U1.IO21
- new net ACIN: ACIN/OUT-2.KL, K2.COM
- new net AMP_METER/IN: IC1.I-_0, IC1.I-_1, K2.NO
- new net AMP_METER/OUT: ACIN/OUT-1.KL, IC1.I+_0, IC1.I+_1
- new net DELETE: C3.2, IC1.FILTER
- new net GPIO05: JP1.4, U1.IO5
- new net GPIO17: JP1.6, U1.IO17
- new net GPIO18: JP1.2, U1.IO18
- new net GPIO19: JP1.3, U1.IO19
- new net GPIO21: JP1.1, U1.IO21
- new net N$12: K1.NO, VALVESOLENOID_01-1.KL
- new net N$14: R2.1, R3.2, U3.ET
- new net N$16: Q3.B, R4.2
- new net N$18: R4.1, R8.2, U4.ET
- new net N$20: K4.COM, VALVESOLENOID_03-2.KL
- new net N$22: R6.1, U$1.A
- new net N$24: K4.NO, VALVESOLENOID_03-1.KL
- new net N$28: JP2.3
- new net N$43: Q1.B, R1.2
- new net N$7: Q2.B, R2.2
- new net N$8: R11.1, U$5.A
- new net PUMPRELAYSEGMENT: D1.A, K2.A2, Q1.C
- new net RELAY1SEGMENT: D2.A, K1.A2, Q2.C
- new net RELAY2SEGMENT: D3.A, K3.A2, Q3.C
- new net RELAY3SEGMENT: D4.A, K4.A2, Q4.C
- net 3V3: now also R17.1; no longer R10.2
- net DTR: now also R19.2; no longer R22.2
- net GND: now also C3.1, C4.1, IC1.GND, Q1.E, Q2.E, Q3.E, Q4.E, U$4.C, U2.C, U3.C, U4.C, U5.C; no longer GND1-1.KL, SC_00-1.KL, SC_01-1.KL, SC_02-1.KL, SC_03-1.KL, SC_04-1.KL, SC_05-1.KL, SC_06-1.KL, SC_07-1.KL, SC_08-1.KL, U$11.C, U$12.C, U$13.C, U$14.C, U$15.C, U$16.C, U$8.C
- net GPIO0: now also R17.2
- net GPIO12: now also JP2.4
- net GPIO13/PUMP_RELAY: now also U2.A; no longer R4.2, SC_00-3.KL
- net GPIO14: now also JP2.2
- net GPIO16/CURRENT_SENSE: now also IC1.VOUT; no longer GND1-3.KL, R2.2
- net GPIO25/VALVE_RELAY01: now also U3.A; no longer R5.2, SC_01-3.KL
- net GPIO26/VALVE_RELAY02: now also U4.A; no longer R6.2, SC_02-3.KL
- net GPIO27/VALVE_RELAY03: now also U5.A; no longer R8.2, SC_03-3.KL
- net GPIO34/DHT: no longer U$6.DAT
- net GPIO36: now also JP2.5
- net GPIO39: now also JP2.6
- net GPIO4: now also R16.2; no longer R11.2, SC_04-3.KL
- net N$13: now also R3.1, U$3.A; no longer R4.1, U$5.A
- net N$15: now also K3.COM, VALVESOLENOID_02-2.KL; no longer R5.1, U$7.A
- net N$17: now also R8.1, U$4.A; no longer R6.1, U$8.A
- net N$19: now also K3.NO, VALVESOLENOID_02-1.KL; no longer R8.1, U$11.A
- net N$2: now also R11.2, U2.ET; no longer U$1.A
- net N$21: now also Q4.B, R5.2; no longer R11.1, U$12.A
- net N$23: now also R5.1, R6.2, U5.ET; no longer R16.1, U$13.A
- net N$26: now also R10.2, U$6.DAT; no longer Q5.B, R21.1
- net N$27: now also JP2.1; no longer R17.1, U$14.A
- net N$29: now also R16.1, U$7.A; no longer R18.1, U$15.A
- net N$31: now also Q5.B, R18.1; no longer R19.1, U$16.A
- net N$34: now also R19.1; no longer R22.1
- net N$5: now also K1.COM, VALVESOLENOID_01-2.KL; no longer R2.1, U$3.A
- net RTS: now also R18.2; no longer R21.2
- net VCC: now also C4.2, D1.C, D2.C, D3.C, D4.C, IC1.VCC, K1.A1, K2.A1, K3.A1, K4.A1, U2.CT, U3.CT, U4.CT, U5.CT; no longer GND1-2.KL, SC_00-2.KL, SC_01-2.KL, SC_02-2.KL, SC_03-2.KL, SC_04-2.KL, SC_05-2.KL, SC_06-2.KL, SC_07-2.KL, SC_08-2.KL
Other:
- moved on the sheet: Q5, Q6, R1, R10, R11, R16, R17, R18, R19, R2, R4, R5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
