File: pcb/2.0/esplash.brd (EAGLE design)
At the start: 72 x 102 mm, 57 parts, among them Q5 BCX70SMD, Q6 BCX70SMD, U1 ESP-WROOM-32, Y1 ECS-.327-12.5-13X

Commit message: change to battery sensing board
Parts:
- removed GND1, SC_08: SC, con-wago-500:W237-103
- removed R11, R13, R16, R17, R18, R19: 100ohm, fab:R1206
- removed U$11, U$12, U$13, U$14, U$15, U$16, U$3, U$5, U$7, U$8, U$9: LED, fab:LED1206
- removed U$2: MCP1700T-3302E/TT, MCP1700T-3302E_TT:SOT95P237X112-3N
- removed U$6: TEMP-HUM-SENSOR-DHT11, diy-modules:TEMP-HUM-SENSOR-DHT11
- added C3, C4: 1uF, fab:C1206FAB
- added R20, R3: 50 ohm, fab:R1206
- C1: value 100nF -> 10uF
- C2: value 100uF -> 100nF
- R1, R6, R8: value 100ohm -> 10Kohm; device fab:R1206 -> fab:R1206FAB
- R10: value 10K -> 5Kohm
- R15: value 10k -> 5M
- R4: value 100ohm -> 100Kohm; device fab:R1206 -> fab:R1206FAB
- R5: value 100ohm -> 4.9Kohm; device fab:R1206 -> fab:R1206FAB
- R7: value 1.2Mohm -> 49.9Kohm
- R9: value 1.5Mohm -> 50Kohm
- moved SC_07 230.8 mm to (-16.7, -125.9), turned to 0 degrees
- moved R8 184.5 mm to (-21.9, -147.7), turned to 0 degrees
- moved U$1 181.2 mm to (-21.8, -91.4), turned to 0 degrees
- moved R6 168.9 mm to (-21.9, -142.1), turned to 0 degrees
- moved R2 168.8 mm to (-21.8, -85.3), turned to 0 degrees
- moved R4 161.3 mm to (-21.9, -108.3), turned to 0 degrees
- moved R5 159.4 mm to (-21.9, -136.6), turned to 0 degrees
- moved R10 156.6 mm to (-21.9, -119.3), turned to 0 degrees
- moved R1 154.4 mm to (-21.9, -68.3), turned to 0 degrees
- moved R9 142.9 mm to (-21.9, -113.8), turned to 0 degrees
- moved C2 94.8 mm to (-21.9, -79.4)
- moved C1 93.3 mm to (-21.9, -73.9), turned to 0 degrees
Connections:
- removed net GPIO05/VALVE_RELAY07: R18.2, SC_07.3, U1.29
- removed net GPIO12: U1.14
- removed net GPIO13/PUMP_RELAY: R4.2, SC_00.3, U1.16
- removed net GPIO14: U1.13
- removed net GPIO16/CURRENT_SENSE: GND1.3, R2.2, U1.27
- removed net GPIO17/VALVE_RELAY08: R19.2, SC_08.3, U1.28
- removed net GPIO18/VALVE_RELAY06: R17.2, SC_06.3, U1.30
- removed net GPIO19/VALVE_RELAY05: R16.2, SC_05.3, U1.31
- removed net GPIO21/VALVE_RELAY04: R1.2, U1.33
- removed net GPIO25/VALVE_RELAY01: R5.2, SC_01.3, U1.10
- removed net GPIO26/VALVE_RELAY02: R6.2, SC_02.3, U1.11
- removed net GPIO27/VALVE_RELAY03: R8.2, SC_03.3, U1.12
- removed net GPIO34/DHT: R10.1, U$6.2, U1.6
- removed net GPIO35/BATTVOLT: R7.1, R9.2, U1.7
- removed net GPIO4: R11.2, SC_04.3, U1.26
- removed net N$13: R4.1, U$5.1
- removed net N$15: R5.1, U$7.1
- removed net N$17: R6.1, U$8.1
- removed net N$19: R8.1, U$11.1
- removed net N$21: R11.1, U$12.1
- removed net N$23: R16.1, U$13.1
- removed net N$25: R13.1, U$9.1
- removed net N$27: R17.1, U$14.1
- removed net N$29: R18.1, U$15.1
- removed net N$31: R19.1, U$16.1
- new net BUT_CHIP_LO: R20.1, S1.3, S1.4
- new net BUT_IO0_LO: R3.1, S2.3, S2.4
- new net GPIO05: U1.29
- new net GPIO12/BATT_IN_7: SC_06.3, U1.14
- new net GPIO13/BATT_IN_8: SC_07.3, U1.16
- new net GPIO14/BATT_IN_6: SC_05.3, U1.13
- new net GPIO16: U1.27
- new net GPIO17: U1.28
- new net GPIO18: U1.30
- new net GPIO19: U1.31
- new net GPIO21: U1.33
- new net GPIO25/BATT_IN_3: SC_02.3, U1.10
- new net GPIO26/BATT_IN_4: SC_03.3, U1.11
- new net GPIO27/BATT_IN_5: SC_04.3, U1.12
- new net GPIO34/BATT_IN_1: SC_00.3, U1.6
- new net GPIO35/BATT_IN_2: SC_01.3, U1.7
- new net GPIO4/POWER_VOLT_IN: R1.2, R10.1, U1.26
- new net N$12: R5.2
- new net N$3: R4.2, R7.1, R9.2
- new net N$6: R5.1, R6.2
- new net N$7: R6.1, R8.2
- new net N$8: R8.1
- net 3V3: now also C3.1, R2.2; no longer R10.2, R13.2, U$2.2, U$6.1
- net CHIP_PU: now also C4.1
- net GND: now also C3.2, C4.2, R1.1, R20.2, R3.2; no longer GND1.1, R9.1, S1.3, S1.4, S2.3, S2.4, SC_08.1, U$11.2, U$12.2, U$13.2, U$14.2, U$15.2, U$16.2, U$2.1, U$3.2, U$5.2, U$6.4, U$7.2, U$8.2, U$9.2
- net N$2: now also R2.1; no longer R1.1
- net N$5: now also R10.2, R4.1, R9.1; no longer R2.1, U$3.1
- net VCC: no longer GND1.2, SC_08.2, U$2.3
Routing:
- net GPIO26/VALVE_RELAY02: track 68.7 -> 0.00 mm
- net GPIO4: track 66.2 -> 0.00 mm
- net GPIO25/VALVE_RELAY01: track 59.2 -> 0.00 mm
- net GPIO4/POWER_VOLT_IN: track 0.00 -> 56.3 mm
- net GPIO27/VALVE_RELAY03: track 55.5 -> 0.00 mm
- net GPIO16/CURRENT_SENSE: track 53.2 -> 0.00 mm
- net GPIO17/VALVE_RELAY08: track 52.4 -> 0.00 mm
- net GPIO13/PUMP_RELAY: track 51.4 -> 0.00 mm
- net GPIO05/VALVE_RELAY07: track 49.1 -> 0.00 mm
- net GPIO19/VALVE_RELAY05: track 47.2 -> 0.00 mm
- net GPIO19: track 0.00 -> 45.4 mm
- net GPIO18/VALVE_RELAY06: track 42.3 -> 0.00 mm
- net GPIO17: track 0.00 -> 41.5 mm
- net GPIO27/BATT_IN_5: track 0.00 -> 40.8 mm
- net GPIO26/BATT_IN_4: track 0.00 -> 40.6 mm
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