File: pcb/2.0/esplash.sch (EAGLE design)
At the start: 57 parts, among them Q5 BCX70SMD, Q6 BCX70SMD, U1 ESP-WROOM-32, Y1 ECS-.327-12.5-13X

Commit message: change to battery sensing board
Parts:
- removed GND1, SC_08: SC, con-wago-500:W237-103
- removed R11, R13, R16, R17, R18, R19: 100ohm, fab:RES-US1206
- removed U$11, U$12, U$13, U$14, U$15, U$16, U$3, U$5, U$7, U$8, U$9: LED, fab:LED
- removed U$2: MCP1700T-3302E/TT, MCP1700T-3302E_TT:MCP1700T-3302E/TT
- removed U$6: TEMP-HUM-SENSOR-DHT11, diy-modules:TEMP-HUM-SENSOR-DHT11
- added C3, C4: 1uF, fab:CAP-UNPOLARIZEDFAB
- added R20, R3: 50 ohm, fab:RES-US1206
- C1: value 100nF -> 10uF
- C2: value 100uF -> 100nF; device fab:CAP-US1206FAB -> fab:CAP-UNPOLARIZEDFAB
- R1, R6, R8: value 100ohm -> 10Kohm; device fab:RES-US1206 -> fab:RES-US1206FAB
- R10: value 10K -> 5Kohm
- R15: value 10k -> 5M
- R4: value 100ohm -> 100Kohm; device fab:RES-US1206 -> fab:RES-US1206FAB
- R5: value 100ohm -> 4.9Kohm; device fab:RES-US1206 -> fab:RES-US1206FAB
- R7: value 1.2Mohm -> 49.9Kohm
- R9: value 1.5Mohm -> 50Kohm
Connections:
- removed net GPIO05/VALVE_RELAY07: R18.2, SC_07-3.KL, U1.IO5
- removed net GPIO12: U1.IO12
- removed net GPIO13/PUMP_RELAY: R4.2, SC_00-3.KL, U1.IO13
- removed net GPIO14: U1.IO14
- removed net GPIO16/CURRENT_SENSE: GND1-3.KL, R2.2, U1.IO16
- removed net GPIO17/VALVE_RELAY08: R19.2, SC_08-3.KL, U1.IO17
- removed net GPIO18/VALVE_RELAY06: R17.2, SC_06-3.KL, U1.IO18
- removed net GPIO19/VALVE_RELAY05: R16.2, SC_05-3.KL, U1.IO19
- removed net GPIO21/VALVE_RELAY04: R1.2, U1.IO21
- removed net GPIO25/VALVE_RELAY01: R5.2, SC_01-3.KL, U1.IO25
- removed net GPIO26/VALVE_RELAY02: R6.2, SC_02-3.KL, U1.IO26
- removed net GPIO27/VALVE_RELAY03: R8.2, SC_03-3.KL, U1.IO27
- removed net GPIO34/DHT: R10.1, U$6.DAT, U1.IO34
- removed net GPIO35/BATTVOLT: R7.1, R9.2, U1.IO35
- removed net GPIO4: R11.2, SC_04-3.KL, U1.IO4
- removed net N$13: R4.1, U$5.A
- removed net N$15: R5.1, U$7.A
- removed net N$17: R6.1, U$8.A
- removed net N$19: R8.1, U$11.A
- removed net N$21: R11.1, U$12.A
- removed net N$23: R16.1, U$13.A
- removed net N$25: R13.1, U$9.A
- removed net N$27: R17.1, U$14.A
- removed net N$29: R18.1, U$15.A
- removed net N$31: R19.1, U$16.A
- new net BUT_CHIP_LO: R20.1, S1.S, S1.S1
- new net BUT_IO0_LO: R3.1, S2.S, S2.S1
- new net GPIO05: U1.IO5
- new net GPIO12/BATT_IN_7: SC_06-3.KL, U1.IO12
- new net GPIO13/BATT_IN_8: SC_07-3.KL, U1.IO13
- new net GPIO14/BATT_IN_6: SC_05-3.KL, U1.IO14
- new net GPIO16: U1.IO16
- new net GPIO17: U1.IO17
- new net GPIO18: U1.IO18
- new net GPIO19: U1.IO19
- new net GPIO21: U1.IO21
- new net GPIO25/BATT_IN_3: SC_02-3.KL, U1.IO25
- new net GPIO26/BATT_IN_4: SC_03-3.KL, U1.IO26
- new net GPIO27/BATT_IN_5: SC_04-3.KL, U1.IO27
- new net GPIO34/BATT_IN_1: SC_00-3.KL, U1.IO34
- new net GPIO35/BATT_IN_2: SC_01-3.KL, U1.IO35
- new net GPIO4/POWER_VOLT_IN: R1.2, R10.1, U1.IO4
- new net N$12: R5.2
- new net N$3: R4.2, R7.1, R9.2
- new net N$6: R5.1, R6.2
- new net N$7: R6.1, R8.2
- new net N$8: R8.1
- net 3V3: now also C3.1, R2.2; no longer R10.2, R13.2, U$2.VOUT, U$6.VDD
- net CHIP_PU: now also C4.1
- net GND: now also C3.2, C4.2, R1.1, R20.2, R3.2; no longer GND1-1.KL, R9.1, S1.S, S1.S1, S2.S, S2.S1, SC_08-1.KL, U$11.C, U$12.C, U$13.C, U$14.C, U$15.C, U$16.C, U$2.GND, U$3.C, U$5.C, U$6.GND, U$7.C, U$8.C, U$9.C
- net N$2: now also R2.1; no longer R1.1
- net N$5: now also R10.2, R4.1, R9.1; no longer R2.1, U$3.A
- net VCC: no longer GND1-2.KL, SC_08-2.KL, U$2.VIN
Other:
- note added: "Automatic Reset"
- note added: "Battery Connections"
- note added: "Crystal"
- note added: "Decoupling Caps"
- note removed: "Current Sensor"
- note removed: "Humidity Sensor"
- note removed: "RELAYS"
- moved on the sheet: C1, C5, C6, Q5, Q6, R1, R10, R12, R14, R15, R2, R21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

Commit message: Finished PCB
Parts:
- added R11, R30, R32: 4.9Kohm, fab:RES-US1206FAB
- added R13, R18, R25, R29, R33, R37, R41, R45: 49.9Kohm, fab:RES-US1206FAB
- added R16, R19, R23, R26, R31, R34, R35, R38, R39, R42: 10Kohm, fab:RES-US1206FAB
- added R17, R27, R36, R44: 100Kohm, fab:RES-US1206FAB
- added R24, R28, R40, R43: 4.99Kohm, fab:RES-US1206FAB
Connections:
- new net N$13: R8.1, SC_00-1.KL
- new net N$14: R11.2, SC_01-3.KL
- new net N$15: R11.1, R13.2, R17.2
- new net N$16: R23.1, SC_02-1.KL
- new net N$17: R18.1, R19.2
- new net N$18: R19.1, R24.2
- new net N$19: R25.2, SC_03-3.KL
- new net N$20: R25.1, R27.2, R29.2
- new net N$21: R26.1, SC_03-1.KL
- new net N$22: R27.1, R28.2, R29.1
- new net N$23: R30.1, R31.2
- new net N$24: R30.2, SC_04-3.KL
- new net N$25: R32.2, SC_05-3.KL
- new net N$27: R34.1, SC_05-1.KL
- new net N$28: R35.1, SC_04-1.KL
- new net N$29: R32.1, R33.2, R36.2
- new net N$30: R37.2, SC_06-3.KL
- new net N$31: R37.1, R39.2
- new net N$32: R38.1, SC_06-1.KL
- new net N$33: R39.1, R40.2
- new net N$35: R41.2, SC_07-3.KL
- new net N$36: R41.1, R44.2, R45.2
- new net N$37: R43.2, R44.1, R45.1
- new net N$38: R42.1, SC_07-1.KL
- net GND: no longer SC_00-1.KL, SC_01-1.KL, SC_02-1.KL, SC_03-1.KL, SC_04-1.KL, SC_05-1.KL, SC_06-1.KL, SC_07-1.KL
- net GPIO12/BATT_IN_7: now also R38.2, R40.1; no longer SC_06-3.KL
- net GPIO13/BATT_IN_8: now also R42.2, R43.1; no longer SC_07-3.KL
- net GPIO14/BATT_IN_6: now also R33.1, R34.2, R36.1; no longer SC_05-3.KL
- net GPIO25/BATT_IN_3: now also R23.2, R24.1; no longer SC_02-3.KL
- net GPIO26/BATT_IN_4: now also R26.2, R28.1; no longer SC_03-3.KL
- net GPIO27/BATT_IN_5: now also R31.1, R35.2; no longer SC_04-3.KL
- net GPIO34/BATT_IN_1: now also R6.1, R8.2; no longer SC_00-3.KL
- net GPIO35/BATT_IN_2: now also R13.1, R16.2, R17.1; no longer SC_01-3.KL
- net N$12: now also SC_00-3.KL
- net N$7: now also R18.2, SC_02-3.KL; no longer R6.1, R8.2
- net N$8: now also R16.1, SC_01-1.KL; no longer R8.1
- net VCC: no longer SC_00-2.KL, SC_01-2.KL, SC_02-2.KL, SC_03-2.KL, SC_04-2.KL, SC_05-2.KL, SC_06-2.KL, SC_07-2.KL
Other:
- note added: "Automatic Programming"
- note removed: "Automatic Reset"
- moved on the sheet: R5, R6, R8, SC_00-1, SC_00-2, SC_00-3, SC_01-1, SC_01-2, SC_01-3, SC_02-1, SC_02-2, SC_02-3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
