File: pcb/1.0 Backup/esplash.sch (EAGLE design)
At the start: 57 parts, among them Q5 BCX70SMD, Q6 BCX70SMD, U1 ESP-WROOM-32, Y1 ECS-.327-12.5-13X

Commit message: Finished PCB
Parts:
- removed GND1, SC_00, SC_01, SC_02, SC_03, SC_04, SC_05, SC_06, SC_07, SC_08: SC, con-wago-500:W237-103
- removed R11, R13, R16, R17, R18, R19: 100ohm, fab:RES-US1206
- removed R15: 10k, fab:RES-US1206
- removed U$11, U$12, U$13, U$14, U$15, U$16, U$3, U$5, U$7, U$8, U$9: LED, fab:LED
- removed U$2: MCP1700T-3302E/TT, MCP1700T-3302E_TT:MCP1700T-3302E/TT
- removed U$6: TEMP-HUM-SENSOR-DHT11, diy-modules:TEMP-HUM-SENSOR-DHT11
- added C3, C4: 1uF, fab:CAP-UNPOLARIZEDFAB
- added PAD1, PAD2, PAD3, PAD4: (no value), wirepad:2,15/1,0
- added R111, R211, R511, R611: 4.9Kohm, fab:RES-US1206FAB
- added R121, R131, R231, R321, R341, R441, R521, R531, R631, R721, R741, R841: 10Kohm, fab:RES-US1206FAB
- added R221, R421, R621, R821: 100Kohm, fab:RES-US1206FAB
- added R222, R311, R411, R422, R622, R711, R811, R822: 49.9Kohm, fab:RES-US1206FAB
- added R3: 50ohm, fab:RES-US1206FAB
- added R331, R431, R731, R831: 4.99Kohm, fab:RES-US1206FAB
- added SC_1, SC_2, SC_3, SC_4, SC_5, SC_6, SC_7, SC_8: SC, con-wago-500:W237-103
- C1: value 100nF -> 10uF
- C2: value 100uF -> 100nF; device fab:CAP-US1206FAB -> fab:CAP-UNPOLARIZEDFAB
- R1: value 100ohm -> 49.9Kohm; device fab:RES-US1206 -> fab:RES-US1206FAB
- R10: value 10K -> 0 ohm
- R4: value 100ohm -> 10Kohm; device fab:RES-US1206 -> fab:RES-US1206FAB
- R5: value 100ohm -> 100Kohm; device fab:RES-US1206 -> fab:RES-US1206FAB
- R6: value 100ohm -> 50Kohm; device fab:RES-US1206 -> fab:RES-US1206FAB
- R7: value 1.2Mohm -> 50ohm
- R8: value 100ohm -> 5Kohm; device fab:RES-US1206 -> fab:RES-US1206FAB
- R9: value 1.5Mohm -> 0 ohm
- renumbered POWER to POWER1
Connections:
- removed net GPIO05/VALVE_RELAY07: R18.2, SC_07-3.KL, U1.IO5
- removed net GPIO12: U1.IO12
- removed net GPIO13/PUMP_RELAY: R4.2, SC_00-3.KL, U1.IO13
- removed net GPIO14: U1.IO14
- removed net GPIO15: U1.IO15
- removed net GPIO16/CURRENT_SENSE: GND1-3.KL, R2.2, U1.IO16
- removed net GPIO17/VALVE_RELAY08: R19.2, SC_08-3.KL, U1.IO17
- removed net GPIO18/VALVE_RELAY06: R17.2, SC_06-3.KL, U1.IO18
- removed net GPIO19/VALVE_RELAY05: R16.2, SC_05-3.KL, U1.IO19
- removed net GPIO21/VALVE_RELAY04: R1.2, U1.IO21
- removed net GPIO22: U1.IO22
- removed net GPIO23: U1.IO23
- removed net GPIO25/VALVE_RELAY01: R5.2, SC_01-3.KL, U1.IO25
- removed net GPIO26/VALVE_RELAY02: R6.2, SC_02-3.KL, U1.IO26
- removed net GPIO27/VALVE_RELAY03: R8.2, SC_03-3.KL, U1.IO27
- removed net GPIO34/DHT: R10.1, U$6.DAT, U1.IO34
- removed net GPIO35/BATTVOLT: R7.1, R9.2, U1.IO35
- removed net GPIO36: U1.SENSOR_VP
- removed net GPIO39: U1.SENSOR_VN
- removed net GPIO4: R11.2, SC_04-3.KL, U1.IO4
- removed net N$15: R5.1, U$7.A
- removed net N$17: R6.1, U$8.A
- removed net N$23: R16.1, U$13.A
- removed net N$25: R13.1, U$9.A
- removed net N$27: R17.1, U$14.A
- removed net N$29: R18.1, U$15.A
- removed net N$31: R19.1, U$16.A
- removed net N$5: R2.1, U$3.A
- new net GPIO12/BATT_IN_7: R731.1, R741.2, U1.IO12
- new net GPIO13/BATT_IN_8: R831.1, R841.2, U1.IO13
- new net GPIO14/BATT_IN_6: R621.1, R622.1, R631.2, U1.IO14
- new net GPIO25/BATT_IN_3: R331.1, R341.2, U1.IO25
- new net GPIO26/BATT_IN_4: R431.1, R441.2, U1.IO26
- new net GPIO27/BATT_IN_5: R521.1, R531.2, U1.IO27
- new net GPIO34/BATT_IN_1: R121.1, R131.2, U1.IO34
- new net GPIO35/BATT_IN_2: R221.1, R222.1, R231.2, U1.IO35
- new net GPIO4/POWER_VOLT_IN: R4.2, R8.1, U1.IO4
- new net N$12: R111.2, SC_1-1.KL
- new net N$14: R211.2, SC_2-1.KL
- new net N$16: R611.2, SC_6-3.KL
- new net N$18: R10.2, R9.1
- new net N$20: R211.1, R221.2, R222.2
- new net N$22: R311.2, SC_3-1.KL
- new net N$24: R311.1, R321.2
- new net N$30: R321.1, R331.2
- new net N$32: R411.2, SC_4-3.KL
- new net N$33: R411.1, R421.2, R422.2
- new net N$35: R421.1, R422.1, R431.2
- new net N$37: R511.1, R521.2
- new net N$38: R511.2, SC_5-3.KL
- new net N$42: R611.1, R621.2, R622.2
- new net N$43: R711.2, SC_7-1.KL
- new net N$44: R711.1, R721.2
- new net N$46: R721.1, R731.2
- new net N$47: R811.2, SC_8-1.KL
- new net N$48: R811.1, R821.2, R822.2
- new net N$49: R821.1, R822.1, R831.2
- new net N$6: R3.2, S1.S, S1.S1
- new net N$8: R111.1, R121.2
- net 32K_XN: no longer R15.2
- net 32K_XP: no longer R15.1
- net 3V3: now also C3.1, PAD3.P, R2.2; no longer R10.2, R13.2, U$2.VOUT, U$6.VDD
- net CHIP_PU: now also C4.1
- net GND: now also C3.2, C4.2, PAD2.P, PAD4.P, R10.1, R131.1, R231.1, R3.1, R341.1, R4.1, R441.1, R531.1, R631.1, R7.1, R741.1, R841.1, R9.2, SC_1-3.KL, SC_2-3.KL, SC_3-3.KL, SC_4-1.KL, SC_5-1.KL, SC_6-1.KL, SC_7-3.KL, SC_8-3.KL; no longer GND1-1.KL, R9.1, S1.S, S1.S1, S2.S, S2.S1, SC_00-1.KL, SC_01-1.KL, SC_02-1.KL, SC_03-1.KL, SC_04-1.KL, SC_05-1.KL, SC_06-1.KL, SC_07-1.KL, SC_08-1.KL, U$11.C, U$12.C, U$13.C, U$14.C, U$15.C, U$16.C, U$2.GND, U$3.C, U$5.C, U$6.GND, U$7.C, U$8.C, U$9.C
- net N$13: now also R5.1, R6.1, R8.2; no longer R4.1, U$5.A
- net N$19: now also R2.1, U$1.A; no longer R8.1, U$11.A
- net N$2: now also R5.2, R6.2; no longer U$1.A
- net N$21: now also R7.2, S2.S, S2.S1; no longer R11.1, U$12.A
- net VCC: now also PAD1.P, R1.2; no longer GND1-2.KL, R7.2, SC_00-2.KL, SC_01-2.KL, SC_02-2.KL, SC_03-2.KL, SC_04-2.KL, SC_05-2.KL, SC_06-2.KL, SC_07-2.KL, SC_08-2.KL, U$2.VIN
Other:
- note added: "Automatic Programming"
- note added: "Battery Connections"
- note added: "Crystal"
- note added: "Decoupling Caps"
- note removed: "Current Sensor"
- note removed: "Humidity Sensor"
- note removed: "RELAYS"
- moved on the sheet: C1, C5, C6, Q5, Q6, R1, R10, R2, R21, R22, R4, R5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
